Commit message: Corrected wheel rotation axe issue

File: urdf/wheel.urdf.xacro (robot description, xacro)
@@ -14,5 +14,5 @@
       <link name="${fb}_${lr}_wheel">
          <visual>
-            <origin xyz="0 0 0" rpy="${flipY*M_PI/2} 0 0"/>  <!-- make sure the wheel is in the correc position -->
+            <origin xyz="0 0 0" rpy="${flipY*M_PI/2} 0 0"/>  <!-- make sure the wheel is in the correct position -->
             <geometry>
                <cylinder length="${wheel_width}" radius="${wheel_radius}" />
@@ -46,4 +46,5 @@
          <origin xyz="${translateX} ${translateY} ${translateZ}" rpy="0 0 0" />
          <limit effort="1000" velocity="1000" />
+         <axis xyz="0 1 0" />
          <joint_properties damping="0.0" friction="0.0" />
       </joint>
@@ -54,5 +55,5 @@
          <actuator name="${fb}_${lr}_wheel_joint_motor">
             <hardwareInterface>EffortJointInterface</hardwareInterface>
-            <mechanicalReduction>1</mechanicalReduction> <!-- It is not true: we uses motor with gearbos and ration of 75 -->
+            <mechanicalReduction>1</mechanicalReduction> <!-- It is not true: we uses motor with gearbox and ration of 75 -->
          </actuator>
       </transmission>

Commit message: Corrected hardware interface

File: urdf/wheel.urdf.xacro (robot description, xacro)
@@ -48,11 +48,14 @@
          <axis xyz="0 1 0" />
          <joint_properties damping="0.0" friction="0.0" />
+         <type>transmission_interface/SimpleTransmission</type>
       </joint>
       <!-- Transmission is important to link the joint and the controller -->
       <transmission name="${fb}_${lr}_wheel_joint_trans" >
          <type>transmission_interface/SimpleTransmission</type>
-         <joint name="${fb}_${lr}_wheel_joint" />
+         <joint name="${fb}_${lr}_wheel_joint">
+            <hardwareInterface>hardware_interface/EffortJointInterface</hardwareInterface>
+         </joint>
          <actuator name="${fb}_${lr}_wheel_joint_motor">
-            <hardwareInterface>EffortJointInterface</hardwareInterface>
+            <hardwareInterface>hardware_interface/EffortJointInterface</hardwareInterface>
             <mechanicalReduction>1</mechanicalReduction> <!-- It is not true: we uses motor with gearbox and ration of 75 -->
          </actuator>
