Commit message: Added joystick node

File: urdf/gribot.xacro (robot description, xacro)
@@ -40,11 +40,11 @@
    <!-- base_footprint is a fictious link(frame) that is on the ground right below base_link origin -->
    <link name="base_footprint">
-      <inertial>
-         <mass value="0.0001" />
-         <origin xyz="0 0 0"  />
-         <inertia ixx="0.0001" ixy="0.0" ixz="0.0"
-               iyy="0.0001" iyz="0.0"
-               izz="0.0001" />
-      </inertial>
+      <!-- <inertial> -->
+         <!-- <mass value="0.0001" /> -->
+         <!-- <origin xyz="0 0 0"  /> -->
+         <!-- <inertia ixx="0.0001" ixy="0.0" ixz="0.0" -->
+         <!--      iyy="0.0001" iyz="0.0" -->
+         <!--      izz="0.0001" /> -->
+      <!-- </inertial> -->
       <visual>
          <origin xzy="0 0 0" rpy="0 0 0" />

Commit message: Added lidar

File: urdf/gribot.xacro (robot description, xacro)
@@ -112,8 +112,65 @@
       </plugin>
    </gazebo>
-<!-- Wheel Definition -->
+   <!-- Wheel Definition -->
    <wheel fb="front" lr="right" parent="base_link" translateX="0.2" translateY="${base_width/2+0.05}"       translateZ="-0.065" flipY="1"/>
    <wheel fb="front" lr="left"  parent="base_link" translateX="0.2" translateY="${-1*(base_width/2+0.05)}"  translateZ="-0.065" flipY="1"/>
    <wheel fb="back"  lr="right" parent="base_link" translateX="-0.2" translateY="${base_width/2+0.05}"      translateZ="-0.065" flipY="1"/>
    <wheel fb="back"  lr="left"  parent="base_link" translateX="-0.2" translateY="${-1*(base_width/2+0.05)}" translateZ="-0.065" flipY="1"/>
+   <!-- Lidar hokuyo -->
+   <link name="lidar_link" >
+      <collision>
+         <origin xyz="0 0 0" rpy="0 0 0" />
+         <geometry>
+            <box size="0.1 0.1 0.1" />
+         </geometry>
+      </collision>
+      <visual>
+         <origin xyz="0 0 0" rpy="0 0 0" />
+         <geometry>
+            <cylinder length="0.1" radius="0.05" />
+         </geometry>
+         <material name="black" />
+      </visual>
+      <inertial>
+         <mass value="1e-5" />
+         <origin xyz="0 0 0" rpy="0 0 0" />
+         <inertia ixx="1e-6" ixy="0" ixz="0" iyy="1e-6" iyz="0" izz="1e-6" />
+      </inertial>
+   </link>
+   <joint name="lidat_to_base" type="fixed" >
+      <origin xyz="0 0 ${base_height/2+0.05}" rpy="0 0 0" />
+      <parent link="base_link" />
+      <child link="lidar_link" />
+   </joint>
+   <gazebo reference="lidar_link" >
+      <sensor type="gpu_ray" name="lidar_sensor">
+         <pose>0 0 0 0 0 0</pose>
+         <visualize>false</visualize>
+         <update_rate>40</update_rate>
+         <ray>
+            <scan>
+               <horizontal>
+                  <samples>720</samples>
+                  <resolution>1</resolution>
+                  <min_angle>-1.570796</min_angle>
+                  <max_angle>1.570796</max_angle>
+               </horizontal>
+            </scan>
+            <range>
+               <min>0.10</min>
+               <max>30.0</max>
+               <resolution>0.01</resolution>
+            </range>
+            <noise>
+               <type>gaussian</type>  <!-- Add parameters for Svcansee sweep -->
+               <mean>0.0</mean>
+               <stddev>0.01</stddev>
+            </noise>
+         </ray>
+         <plugin name="gazebo_ros_head_hokuyo_controller" filename="libgazebo_ros_gpu_laser.so">
+            <topicName>/robot/laser/scan</topicName>
+            <frameName>lidar_link</frameName>
+         </plugin>
+      </sensor>
+   </gazebo>
 </robot>

Commit message: Simplified base_link description

File: urdf/gribot.xacro (robot description, xacro)
@@ -40,17 +40,4 @@
    <!-- base_footprint is a fictious link(frame) that is on the ground right below base_link origin -->
    <link name="base_footprint">
-      <!-- <inertial> -->
-         <!-- <mass value="0.0001" /> -->
-         <!-- <origin xyz="0 0 0"  /> -->
-         <!-- <inertia ixx="0.0001" ixy="0.0" ixz="0.0" -->
-         <!--      iyy="0.0001" iyz="0.0" -->
-         <!--      izz="0.0001" /> -->
-      <!-- </inertial> -->
-      <visual>
-         <origin xzy="0 0 0" rpy="0 0 0" />
-         <geometry>
-            <box size="0.001 0.001 0.001" />
-         </geometry>
-      </visual>
    </link>
    <gazebo reference="base_footprint">

Commit message: Updated joint name for clarification

File: urdf/gribot.xacro (robot description, xacro)
@@ -44,5 +44,5 @@
       <turnGravityOff>false</turnGravityOff>
    </gazebo>
-   <joint name="base_footprint_joint" type="fixed">
+   <joint name="glue_robot_to_world" type="fixed">
       <origin xyz="0 0 0.1" rpy="0 0 0" />
       <parent link="base_footprint" />

Commit message: changed name of base footprint link for clarification

File: urdf/gribot.xacro (robot description, xacro)
@@ -37,14 +37,14 @@
                izz="${0.0833333 * m * (x*x + y*y)}" />
    </xacro:macro>
-   <!-- Base footprint -->
-   <!-- base_footprint is a fictious link(frame) that is on the ground right below base_link origin -->
-   <link name="base_footprint">
+   <!-- World link -->
+   <!-- world_link is a fictious link(frame) that is on the ground right below base_link origin -->
+   <link name="world_link">
    </link>
-   <gazebo reference="base_footprint">
+   <gazebo reference="world_link">
       <turnGravityOff>false</turnGravityOff>
    </gazebo>
    <joint name="glue_robot_to_world" type="fixed">
       <origin xyz="0 0 0.1" rpy="0 0 0" />
-      <parent link="base_footprint" />
+      <parent link="world_link" />
       <child link="base_link" />
    </joint>

Commit message: corrected joint name typo

File: urdf/gribot.xacro (robot description, xacro)
@@ -125,5 +125,5 @@
       </inertial>
    </link>
-   <joint name="lidat_to_base" type="fixed" >
+   <joint name="lidar_to_base" type="fixed" >
       <origin xyz="0 0 ${base_height/2+0.05}" rpy="0 0 0" />
       <parent link="base_link" />

Commit message: Corrected joint typo and updated comments

File: urdf/gribot.xacro (robot description, xacro)
@@ -2,5 +2,5 @@
 <robot name="gribot" xmlns:xacro="http://www.ros.org/wiki/xacro">
    <xacro:include filename="$(find gribot)/urdf/wheel.urdf.xacro" />
-<!-- Defining the colors used in this robot -->
+   <!-- Defining the colors used in this robot -->
    <material name="Black">
       <color rgba="0.0 0.0 0.0 1.0"/>
@@ -76,5 +76,5 @@
       <turnGravityOff>false</turnGravityOff>
    </gazebo>
-   <!-- Skid Steering Drive for 4 wheel robot -->
+   <!-- Skid Steering Drive for 4 wheel robot for simulation -->
    <gazebo>
       <plugin name="skid_steer_drive_controller" filename="libgazebo_ros_skid_steer_drive.so">
@@ -99,10 +99,10 @@
       </plugin>
    </gazebo>
-   <!-- Wheel Definition -->
+   <!-- Wheel Definition for simulation -->
    <wheel fb="front" lr="right" parent="base_link" translateX="0.2" translateY="${base_width/2+0.05}"       translateZ="-0.065" flipY="1"/>
    <wheel fb="front" lr="left"  parent="base_link" translateX="0.2" translateY="${-1*(base_width/2+0.05)}"  translateZ="-0.065" flipY="1"/>
    <wheel fb="back"  lr="right" parent="base_link" translateX="-0.2" translateY="${base_width/2+0.05}"      translateZ="-0.065" flipY="1"/>
    <wheel fb="back"  lr="left"  parent="base_link" translateX="-0.2" translateY="${-1*(base_width/2+0.05)}" translateZ="-0.065" flipY="1"/>
-   <!-- Lidar -->
+   <!-- Lidar definition for simulation -->
    <link name="lidar_link" >
       <collision>
@@ -125,5 +125,5 @@
       </inertial>
    </link>
-   <joint name="lidat_to_base" type="fixed" >
+   <joint name="lidar_to_base" type="fixed" >
       <origin xyz="0 0 ${base_height/2+0.05}" rpy="0 0 0" />
       <parent link="base_link" />
@@ -163,4 +163,5 @@
       </sensor>
    </gazebo>
+   <!-- Publishing joint states from Gazebo simulator -->
    <gazebo>
       <plugin name="joint_state_publisher" filename="libgazebo_ros_joint_state_publisher.so">

Commit message: Configured for gmapping

File: urdf/gribot.xacro (robot description, xacro)
@@ -39,4 +39,6 @@
    <!-- World link -->
    <!-- world_link is a fictious link(frame) that is on the ground right below base_link origin -->
+   <!-- It is necessary as gazebo does not support inertia for the root link -->
+   <!-- Do not call it world as it is reserved for robot that must be fixed to the world -->
    <link name="world_link">
    </link>
@@ -78,5 +80,5 @@
    <!-- Skid Steering Drive for 4 wheel robot for simulation -->
    <gazebo>
-      <plugin name="skid_steer_drive_controller" filename="libgazebo_ros_skid_steer_drive.so">
+      <plugin name="drive_controller" filename="libgazebo_ros_skid_steer_drive.so">
          <updateRate>100</updateRate>
          <robotNameSpace>/</robotNameSpace>
@@ -90,11 +92,11 @@
          <torque>10</torque>
          <topicName>cmd_vel</topicName>
-         <broadcastTF>false</broadcastTF>
-         <commandTopic>cmd_vel</commandTopic>      <!-- default to avoid warning -->
-         <odometryTopic>odom</odometryTopic>       <!-- default to avoid warning -->
-         <odometryFrame>odom</odometryFrame>       <!-- default to avoid warning -->
-         <covariance_x>0.00100</covariance_x>      <!-- default to avoid warning -->
-         <covariance_y>0.00100</covariance_y>      <!-- default to avoid warning -->
-         <covariance_yaw>0.010000</covariance_yaw> <!-- default to avoid warning -->
+         <broadcastTF>true</broadcastTF>  <!-- Must be true or gmapping does not work in simulation environment -->
+         <commandTopic>cmd_vel</commandTopic>
+         <odometryTopic>odom</odometryTopic>
+         <odometryFrame>odom</odometryFrame>
+         <covariance_x>0.00100</covariance_x>
+         <covariance_y>0.00100</covariance_y>
+         <covariance_yaw>0.010000</covariance_yaw>
       </plugin>
    </gazebo>
@@ -105,5 +107,5 @@
    <wheel fb="back"  lr="left"  parent="base_link" translateX="-0.2" translateY="${-1*(base_width/2+0.05)}" translateZ="-0.065" flipY="1"/>
    <!-- Lidar definition for simulation -->
-   <link name="lidar_link" >
+   <link name="sweep_link" >
       <collision>
          <origin xyz="0 0 0" rpy="0 0 0" />
@@ -128,10 +130,10 @@
       <origin xyz="0 0 ${base_height/2+0.05}" rpy="0 0 0" />
       <parent link="base_link" />
-      <child link="lidar_link" />
+      <child link="sweep_link" />
    </joint>
-   <gazebo reference="lidar_link" >
-      <sensor type="ray" name="lidar_sensor">
+   <gazebo reference="sweep_link" >
+      <sensor type="ray" name="laser">
          <pose>0 0 0 0 0 0</pose>
-         <visualize>true</visualize>
+         <visualize>false</visualize>	<!-- temporary for testing, but should be put to false -->
          <update_rate>40</update_rate>
          <ray>
@@ -157,15 +159,16 @@
             </noise>
          </ray>
-         <plugin name="gazebo_ros_head_hokuyo_controller" filename="libgazebo_ros_laser.so">
-            <topicName>/robot/laser/scan</topicName>
-            <frameName>lidar_link</frameName>
+         <plugin name="sweep_link" filename="libgazebo_ros_laser.so">
+            <topicName>base_scan</topicName>
+            <frameName>sweep_link</frameName>
          </plugin>
       </sensor>
    </gazebo>
    <!-- Publishing joint states from Gazebo simulator -->
+   <!-- fixed links are not published -->
    <gazebo>
       <plugin name="joint_state_publisher" filename="libgazebo_ros_joint_state_publisher.so">
          <jointName>front_left_wheel_joint, front_right_wheel_joint, back_left_wheel_joint, back_right_wheel_joint</jointName>
-         <robotNameSpace>/</robotNameSpace>
+         <robotNameSpace>/gribot</robotNameSpace>
          <updateRate>100</updateRate>
          <alwaysOn>true</alwaysOn>

Commit message: Changing link name to avoid confugion

File: urdf/gribot.xacro (robot description, xacro)
@@ -39,15 +39,15 @@
    </xacro:macro>
    <!-- World link -->
-   <!-- world_link is a fictious link(frame) that is on the ground right below base_link origin -->
+   <!-- base_footprint is a fictious link(frame) that is on the ground right below base_link origin -->
    <!-- It is necessary as gazebo does not support inertia for the root link -->
    <!-- Do not call it world as it is reserved for robot that must be fixed to the world -->
-   <link name="world_link">
+   <link name="base_footprint">
    </link>
-   <gazebo reference="world_link">
+   <gazebo reference="base_footprint">
       <turnGravityOff>false</turnGravityOff>
    </gazebo>
    <joint name="glue_robot_to_world" type="fixed">
       <origin xyz="0 0 0.1" rpy="0 0 0" />
-      <parent link="world_link" />
+      <parent link="base_footprint" />
       <child link="base_link" />
    </joint>

Commit message: Changing root link name to avoid confusion

File: urdf/gribot.xacro (robot description, xacro)
@@ -38,15 +38,15 @@
    </xacro:macro>
    <!-- World link -->
-   <!-- world_link is a fictious link(frame) that is on the ground right below base_link origin -->
+   <!-- base_footprint is a fictious link(frame) that is on the ground right below base_link origin -->
    <!-- It is necessary as gazebo does not support inertia for the root link -->
    <!-- Do not call it world as it is reserved for robot that must be fixed to the world -->
-   <link name="world_link">
+   <link name="base_footprint">
    </link>
-   <gazebo reference="world_link">
+   <gazebo reference="base_footprint">
       <turnGravityOff>false</turnGravityOff>
    </gazebo>
    <joint name="glue_robot_to_world" type="fixed">
       <origin xyz="0 0 0.1" rpy="0 0 0" />
-      <parent link="world_link" />
+      <parent link="base_footprint" />
       <child link="base_link" />
    </joint>

Commit message: Navigation is now working, but tuning needs to be applied to navigation. Wheel inversion has been corrected

File: urdf/gribot.xacro (robot description, xacro)
@@ -22,5 +22,5 @@
    <!-- Main body length height width -->
    <xacro:property name="base_height"   value="0.25" /> <!-- in meter -->
-   <xacro:property name="base_width"    value="0.6"  /> <!-- in meter -->
+   <xacro:property name="base_width"    value="0.52"  /> <!-- in meter -->
    <xacro:property name="base_lenght"   value="0.8"  /> <!-- in meter -->
    <xacro:property name="base_mass"     value="20.0" /> <!-- in kg -->
@@ -41,17 +41,17 @@
    <!-- It is necessary as gazebo does not support inertia for the root link -->
    <!-- Do not call it world as it is reserved for robot that must be fixed to the world -->
-   <link name="base_footprint">
+   <link name="base_link">
    </link>
-   <gazebo reference="base_footprint">
+   <gazebo reference="base_link">
       <turnGravityOff>false</turnGravityOff>
    </gazebo>
    <joint name="glue_robot_to_world" type="fixed">
       <origin xyz="0 0 0.1" rpy="0 0 0" />
-      <parent link="base_footprint" />
-      <child link="base_link" />
+      <parent link="base_link" />
+      <child link="chassis" />
    </joint>
    <!-- Base link -->
    <!-- Actual body/chassis of the robot -->
-   <link name="base_link">
+   <link name="chassis">
       <inertial>
          <mass value="${base_mass}" />
@@ -74,5 +74,5 @@
       </collision>
    </link>
-   <gazebo reference="base_link">
+   <gazebo reference="chassis">
       <material>Gazebo/White</material>
       <turnGravityOff>false</turnGravityOff>
@@ -89,5 +89,5 @@
          <wheelSeparation>0.4</wheelSeparation>
          <wheelDiameter>0.32</wheelDiameter>
-         <robotBaseFrame>base_footprint</robotBaseFrame>
+         <robotBaseFrame>base_link</robotBaseFrame>
          <torque>10</torque>
          <topicName>cmd_vel</topicName>
@@ -102,8 +102,8 @@
    </gazebo>
    <!-- Wheel Definition for simulation -->
-   <wheel fb="front" lr="right" parent="base_link" translateX="0.2" translateY="${base_width/2+0.05}"       translateZ="-0.065" flipY="1"/>
-   <wheel fb="front" lr="left"  parent="base_link" translateX="0.2" translateY="${-1*(base_width/2+0.05)}"  translateZ="-0.065" flipY="1"/>
-   <wheel fb="back"  lr="right" parent="base_link" translateX="-0.2" translateY="${base_width/2+0.05}"      translateZ="-0.065" flipY="1"/>
-   <wheel fb="back"  lr="left"  parent="base_link" translateX="-0.2" translateY="${-1*(base_width/2+0.05)}" translateZ="-0.065" flipY="1"/>
+   <wheel fb="front" lr="right" parent="chassis" translateX="0.2" translateY="${-1*(base_width/2+0.04)}"       translateZ="-0.065" flipY="1"/>
+   <wheel fb="front" lr="left"  parent="chassis" translateX="0.2" translateY="${1*(base_width/2+0.04)}"  translateZ="-0.065" flipY="1"/>
+   <wheel fb="back"  lr="right" parent="chassis" translateX="-0.2" translateY="${-1*(base_width/2+0.04)}"      translateZ="-0.065" flipY="1"/>
+   <wheel fb="back"  lr="left"  parent="chassis" translateX="-0.2" translateY="${1*(base_width/2+0.04)}" translateZ="-0.065" flipY="1"/>
    <!-- Lidar definition for simulation -->
    <link name="sweep_link" >
@@ -128,6 +128,6 @@
    </link>
    <joint name="lidar_to_base" type="fixed" >
-      <origin xyz="0 0 ${base_height/2+0.05}" rpy="0 0 0" />
-      <parent link="base_link" />
+      <origin xyz="0.3 0 ${base_height/2+0.05}" rpy="0 0 0" />
+      <parent link="chassis" />
       <child link="sweep_link" />
    </joint>
@@ -136,5 +136,5 @@
          <pose>0 0 0 0 0 0</pose>
          <visualize>false</visualize>	<!-- temporary for testing, but should be put to false -->
-         <update_rate>40</update_rate>
+         <update_rate>100</update_rate> <!-- rate at wich the sensor updates informations -->
          <ray>
             <scan>
@@ -190,14 +190,14 @@
       <!-- </plugin> -->
    <!-- </gazebo> -->
-   <gazebo>
-      <plugin name="imu_plugin" filename="libgazebo_ros_imu.so">
-         <alwaysOn>true</alwaysOn>
-         <bodyName>base_footprint</bodyName>
-         <topicName>imu</topicName>
-         <serviceName>imu_service</serviceName>
-         <gaussianNoise>0.0</gaussianNoise>
-         <updateRate>20.0</updateRate>
-      </plugin>
-   </gazebo>
+   <!-- <gazebo> -->
+      <!-- <plugin name="imu_plugin" filename="libgazebo_ros_imu.so"> -->
+         <!-- <alwaysOn>true</alwaysOn> -->
+         <!-- <bodyName>base_footprint</bodyName> -->
+         <!-- <topicName>imu</topicName> -->
+         <!-- <serviceName>imu_service</serviceName> -->
+         <!-- <gaussianNoise>0.0</gaussianNoise> -->
+         <!-- <updateRate>20.0</updateRate> -->
+      <!-- </plugin> -->
+   <!-- </gazebo> -->
    <gazebo>
       <plugin name="gazebo_ros_control" filename="libgazebo_ros_control.so">
